File: hardware/rev_a/kicad/rev_a.kicad_sch (KiCad schematic)
At the start: 25 parts, among them J2 TSW-110-07-T-D, U1 ADS1299-4PAGR

Commit message: fix(hardware): migrate both bench headers to the high-temperature HTSW selection
Parts:
- J2: value TSW-110-07-T-D -> HTSW-110-07-T-D; MPN TSW-110-07-T-D -> HTSW-110-07-T-D
Changed lines of the file:
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@@
 (in_bom yes) (on_board yes) (dnp no)
 (property "Reference" "J2" (at 43.18 67.31 0) (effects (font (size 1.27 1.27))))
-(property "Value" "TSW-110-07-T-D" (at 43.18 69.85 0) (effects (font (size 1.27 1.27))))
+(property "Value" "HTSW-110-07-T-D" (at 43.18 69.85 0) (effects (font (size 1.27 1.27))))
 (property "Footprint" "Connector_PinHeader_2.54mm:PinHeader_2x10_P2.54mm_Vertical" (at 43.18 99.06 0) (effects (font (size 1.27 1.27)) (hide yes)))
 (property "Datasheet" "" (at 43.18 99.06 0) (effects (font (size 1.27 1.27)) (hide yes)))
 (property "ContractRef" "J_INPUT" (at 43.18 99.06 0) (effects (font (size 1.27 1.27)) (hide yes)))
-(property "MPN" "TSW-110-07-T-D" (at 43.18 99.06 0) (effects (font (size 1.27 1.27)) (hide yes)))
+(property "MPN" "HTSW-110-07-T-D" (at 43.18 99.06 0) (effects (font (size 1.27 1.27)) (hide yes)))
 (property "BOM_ID" "headers" (at 43.18 99.06 0) (effects (font (size 1.27 1.27)) (hide yes)))
 (property "Population" "fit" (at 43.18 99.06 0) (effects (font (size 1.27 1.27)) (hide yes)))
