File: hardware/rev_a/kicad/power.kicad_sch (KiCad schematic)
At the start: 31 parts, among them U1 ADS1299-4PAGR, U2 TPS7A2033PDBVR

Commit message: feat(hardware): publish T491 nominal lands with one fixture pending
The editable local footprints, source/library closure, geometry and courtyard checks, CAD assignments, CSV and tests are published. Remote tree8aa713cd369f7514c97ca628035464c9259c4497 differs from the fully tested local tree4fc3a080680de93b56419376709d76b4b957a0b7 only at tests/fixtures/rev_a_netlist.xml.gz, whose old bytes remain pending transport. Do NOT treat this commit as the full green candidate or merge it.

The clean local2a8c662 candidate passed1051 ordinary+7subtests,98 native/integration,25 actualKiCad cases,1098/1278branches and0ERC findings. Actual native export comparison permits exactly the C_REF/C_VCAP1 footprint IDs, all256 terminals/nets and other component fields unchanged. The pending binary's expected Git blob is a1957d56b6d5db1f6f796066bf275a94d9f908df and raw XML SHA256ca9ccef463e1ab31426ae3afdc9744bd085a6b5bfde18fe231871228ce91fea2. Corrupt orphan uploads were detected by hash checks and never included.

A proposed serialization-helper PR was blocked before any job and its workflow was removed. No write-token transport ran. Fixture projection experiments were also reverted; final local fixture remains the full unmodified native export. Full publication, hosted CI and independent review remain open. All hardware/purchase/body-use gates remain false.
Parts:
- C6: footprint Capacitor_Tantalum_SMD:CP_EIA-7343-31_Kemet-D -> RevA_Passives:T491D_7343_DensityB
- C7: footprint Capacitor_Tantalum_SMD:CP_EIA-3528-21_Kemet-B -> RevA_Passives:T491B_3528_DensityB
Changed lines of the file:
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@@
 (property "Reference" "C6" (at 46.99 144.78 90) (effects (font (size 1.27 1.27))))
 (property "Value" "100u" (at 46.99 148.59 90) (effects (font (size 1.27 1.27))))
-(property "Footprint" "Capacitor_Tantalum_SMD:CP_EIA-7343-31_Kemet-D" (at 38.1 147.32 0) (effects (font (size 1.27 1.27)) (hide yes)))
+(property "Footprint" "RevA_Passives:T491D_7343_DensityB" (at 38.1 147.32 0) (effects (font (size 1.27 1.27)) (hide yes)))
 (property "Datasheet" "" (at 38.1 147.32 0) (effects (font (size 1.27 1.27)) (hide yes)))
 (property "ContractRef" "C_VCAP1" (at 38.1 147.32 0) (effects (font (size 1.27 1.27)) (hide yes)))
@@
 (property "Reference" "C7" (at 143.51 185.42 90) (effects (font (size 1.27 1.27))))
 (property "Value" "22u" (at 143.51 189.23 90) (effects (font (size 1.27 1.27))))
-(property "Footprint" "Capacitor_Tantalum_SMD:CP_EIA-3528-21_Kemet-B" (at 134.62 187.96 0) (effects (font (size 1.27 1.27)) (hide yes)))
+(property "Footprint" "RevA_Passives:T491B_3528_DensityB" (at 134.62 187.96 0) (effects (font (size 1.27 1.27)) (hide yes)))
 (property "Datasheet" "" (at 134.62 187.96 0) (effects (font (size 1.27 1.27)) (hide yes)))
 (property "ContractRef" "C_REF" (at 134.62 187.96 0) (effects (font (size 1.27 1.27)) (hide yes)))

Commit message: feat(hardware): reconstruct routed C4 service access and carrier backing
Parts:
- added J3: B6B-XH-A(LF)(SN), Connector_JST:JST_XH_B6B-XH-A_1x06_P2.50mm_Vertical, symbol RevA:Service_1x06
Connections:
- net AVDD: now also J3.4
- net DVDD: now also J3.2, J3.3
- net GND: now also J3.1, J3.5
- no-connect marks 3 -> 4
Other:
- note added: "C4: auxiliary J104, 1:1 cable. P2 FEED OUT / P3 DVDD SENSE / P4 AVDD SENSE Tie feed and sense at AFE rail only; no powered mating; pin 6 NC. Separate sense is not a Kelvin measurement of the ADC die."
Changed lines of the file:
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@@
 (global_label "GND" (shape passive) (at 238.76 114.3 0) (effects (font (size 1.0 1.0)) (justify left)))
 (sheet_instances (path "/" (page "2")))
+(symbol (lib_id "RevA:Service_1x06") (at 114.3 246.38 0) (unit 1) (exclude_from_sim no) (in_bom yes) (on_board yes) (dnp no)
+(property "Reference" "J3" (at 114.3 228.6 0) (effects (font (size 1.27 1.27)) ))
+(property "Value" "B6B-XH-A(LF)(SN)" (at 114.3 264.16 0) (effects (font (size 1.0 1.0)) ))
+(property "Footprint" "Connector_JST:JST_XH_B6B-XH-A_1x06_P2.50mm_Vertical" (at 124.46 246.38 0) (effects (font (size 1.0 1.0)) (hide yes)))
+(property "Datasheet" "https://www.jst-mfg.com/product/pdf/eng/eXH.pdf" (at 124.46 246.38 0) (effects (font (size 1.0 1.0)) (hide yes)))
+(property "ContractRef" "J_SERVICE" (at 124.46 246.38 0) (effects (font (size 1.0 1.0)) (hide yes)))
+(property "BOM_ID" "service_header" (at 124.46 246.38 0) (effects (font (size 1.0 1.0)) (hide yes)))
+(property "MPN" "B6B-XH-A(LF)(SN)" (at 124.46 246.38 0) (effects (font (size 1.0 1.0)) (hide yes)))
+(property "Population" "fit" (at 124.46 246.38 0) (effects (font (size 1.0 1.0)) (hide yes)))
+(pin "1")
+(pin "2")
+(pin "3")
+(pin "4")
+(pin "5")
+(pin "6")
+(instances (project "rev_a" (path "/6426aeea-facb-56f2-ae10-495fdfe5ecae/bafc1f62-cffb-52cc-860e-95574cf5cdeb" (reference "J3") (unit 1))))
 )
+(wire (pts (xy 93.98 233.68) (xy 104.14 233.68)) (stroke (width 0) (type default)))
+(global_label "GND" (shape input) (at 93.98 233.68 0) (effects (font (size 1 1)) (justify left)) (property "Intersheetrefs" "${INTERSHEET_REFS}" (at 93.98 233.68 0) (effects (font (size 1 1)) (hide yes))))
+(wire (pts (xy 93.98 238.76) (xy 104.14 238.76)) (stroke (width 0) (type default)))
+(global_label "DVDD" (shape input) (at 93.98 238.76 0) (effects (font (size 1 1)) (justify left)) (property "Intersheetrefs" "${INTERSHEET_REFS}" (at 93.98 238.76 0) (effects (font (size 1 1)) (hide yes))))
+(wire (pts (xy 93.98 243.84) (xy 104.14 243.84)) (stroke (width 0) (type default)))
+(global_label "DVDD" (shape input) (at 93.98 243.84 0) (effects (font (size 1 1)) (justify left)) (property "Intersheetrefs" "${INTERSHEET_REFS}" (at 93.98 243.84 0) (effects (font (size 1 1)) (hide yes))))
+(wire (pts (xy 93.98 248.92) (xy 104.14 248.92)) (stroke (width 0) (type default)))
+(global_label "AVDD" (shape input) (at 93.98 248.92 0) (effects (font (size 1 1)) (justify left)) (property "Intersheetrefs" "${INTERSHEET_REFS}" (at 93.98 248.92 0) (effects (font (size 1 1)) (hide yes))))
+(wire (pts (xy 93.98 254) (xy 104.14 254)) (stroke (width 0) (type default)))
+(global_label "GND" (shape input) (at 93.98 254 0) (effects (font (size 1 1)) (justify left)) (property "Intersheetrefs" "${INTERSHEET_REFS}" (at 93.98 254 0) (effects (font (size 1 1)) (hide yes))))
+(no_connect (at 104.14 259.08))
+(text "C4: auxiliary J104, 1:1 cable. P2 FEED OUT / P3 DVDD SENSE / P4 AVDD SENSE\nTie feed and sense at AFE rail only; no powered mating; pin 6 NC.\nSeparate sense is not a Kelvin measurement of the ADC die." (at 30.48 274.32 0) (effects (font (size 1 1)) (justify left)))
+)
