File: hardware/rev_a/auxiliary/auxiliary.kicad_sch (KiCad schematic)
At the start: 8 parts, among them J101 K1_NUMBERED_SOLDER_TAILS, J102 DEVKIT_J1_NUMBERED_TAILS, J103 ADAFRUIT_5335_TAILS, J104 B6B-XH-A(LF)(SN), J105 REGULATED_5V_TAILS, U101 ISO7721DR

Commit message: fix(hardware): update native service note and document exact JST contact suffix
Other:
- note added: "AFE J3 present; use inspected C4 cable."
- note removed: "AFE mating connector/pads NOT YET ADDED."
Changed lines of the file:
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@@
 (text "Port arrows describe external endpoint roles; ERC does not establish power sequencing or physical attachment." (at 15.24 127 0) (effects (font (size 1.27 1.27)) (justify left)))
 (text "J104: dedicated six-way rail access; pin 6 NC." (at 251.46 218.44 0) (effects (font (size 1.27 1.27)) (justify left)))
-(text "AFE mating connector/pads NOT YET ADDED." (at 251.46 223.52 0) (effects (font (size 1.27 1.27)) (justify left)))
+(text "AFE J3 present; use inspected C4 cable." (at 251.46 223.52 0) (effects (font (size 1.27 1.27)) (justify left)))
 (text "HOST_GND and TARGET_GND MUST REMAIN SEPARATE. No host 5-V connection. Both DevKit USBs excluded in acquisition." (at 15.24 246.38 0) (effects (font (size 1.27 1.27)) (justify left)))
 (text "Program bare DevKit before attaching permanent tails. No hot-plugging or small-capacitor-pad flying wires." (at 15.24 254 0) (effects (font (size 1.27 1.27)) (justify left)))
