File: hardware/rev_a/auxiliary/bus.kicad_sch (KiCad schematic)
At the start: 12 parts, among them U102 TXU0304PWR, U103 TXU0304PWR, U104 TXU0304PWR

Commit message: feat(hardware): apply the preserved five-position SPI source candidate
Apply exactly eleven manifest-verified files on 08a8ddd0, retaining
all later DNP, preservation, selection and native-fault test repairs.
The historical patch reproduces 2e50d2b; no geometry is recreated.
Five positions remain DNP/NOT_SELECTED. Native exports and copper
fills are not refreshed here. This is source publication only, not
a passing gate, approved damping value or fabrication release.
No workflow, firmware, Q1, dependency or permission setting changes
are included in this engineering commit. No project code executed
by the isolated source publisher. PR98 must remain draft.
Parts:
- added R117, R118, R119, R120: NOT_SELECTED, Resistor_SMD:R_0603_1608Metric, symbol RevA:R
Connections:
- net AFE_CS: now also R119.2; no longer U102.11 (B3Y)
- net AFE_MOSI: now also R118.2; no longer U102.12 (B2Y)
- net AFE_SCLK: now also R117.2; no longer U102.13 (B1Y)
- net MCU_MISO: now also R120.2; no longer U102.5 (A4Y)
- new net AFE_CS_DRV: R119.1, U102.11 (B3Y)
- new net AFE_MOSI_DRV: R118.1, U102.12 (B2Y)
- new net AFE_SCLK_DRV: R117.1, U102.13 (B1Y)
- new net MCU_MISO_DRV: R120.1, U102.5 (A4Y)
Changed lines of the file:
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@@
 (global_label "MCU_CS" (shape passive) (at 57.15 68.58 180) (effects (font (size 1 1)) (justify right)))
 (wire (pts (xy 60.96 73.66) (xy 57.15 73.66)) (stroke (width 0) (type default)))
-(global_label "MCU_MISO" (shape passive) (at 57.15 73.66 180) (effects (font (size 1 1)) (justify right)))
+(global_label "MCU_MISO_DRV" (shape passive) (at 57.15 73.66 180) (effects (font (size 1 1)) (justify right)))
 (no_connect (at 60.96 78.74))
 (wire (pts (xy 60.96 83.82) (xy 57.15 83.82)) (stroke (width 0) (type default)))
@@
 (global_label "AFE_DVDD" (shape passive) (at 105.41 53.34 0) (effects (font (size 1 1)) (justify left)))
 (wire (pts (xy 101.6 58.42) (xy 105.41 58.42)) (stroke (width 0) (type default)))
-(global_label "AFE_SCLK" (shape passive) (at 105.41 58.42 0) (effects (font (size 1 1)) (justify left)))
+(global_label "AFE_SCLK_DRV" (shape passive) (at 105.41 58.42 0) (effects (font (size 1 1)) (justify left)))
 (wire (pts (xy 101.6 63.5) (xy 105.41 63.5)) (stroke (width 0) (type default)))
-(global_label "AFE_MOSI" (shape passive) (at 105.41 63.5 0) (effects (font (size 1 1)) (justify left)))
+(global_label "AFE_MOSI_DRV" (shape passive) (at 105.41 63.5 0) (effects (font (size 1 1)) (justify left)))
 (wire (pts (xy 101.6 68.58) (xy 105.41 68.58)) (stroke (width 0) (type default)))
-(global_label "AFE_CS" (shape passive) (at 105.41 68.58 0) (effects (font (size 1 1)) (justify left)))
+(global_label "AFE_CS_DRV" (shape passive) (at 105.41 68.58 0) (effects (font (size 1 1)) (justify left)))
 (wire (pts (xy 101.6 73.66) (xy 105.41 73.66)) (stroke (width 0) (type default)))
 (global_label "AFE_MISO" (shape passive) (at 105.41 73.66 0) (effects (font (size 1 1)) (justify left)))
@@
 (wire (pts (xy 339.09 200.66) (xy 342.9 200.66)) (stroke (width 0) (type default)))
 (global_label "TARGET_GND" (shape passive) (at 342.9 200.66 0) (effects (font (size 1 1)) (justify left)))
+(symbol (lib_id "RevA:R") (at 83.82 109.22 0) (unit 1) (in_bom yes) (on_board yes) (dnp yes)
+(property "Reference" "R117" (at 83.82 104.14 0) (effects (font (size 1 1))))
+(property "Value" "NOT_SELECTED" (at 83.82 106.68 0) (effects (font (size 1 1))))
+(property "Footprint" "Resistor_SMD:R_0603_1608Metric" (at 83.82 109.22 0) (effects (font (size 1 1)) (hide yes)))
+(property "Datasheet" "" (at 83.82 109.22 0) (effects (font (size 1 1)) (hide yes)))
+(property "ContractRef" "R_AFE_SCLK_SER" (at 83.82 109.22 0) (effects (font (size 1 1)) (hide yes)))
+(property "MPN" "NOT_SELECTED" (at 83.82 109.22 0) (effects (font (size 1 1)) (hide yes)))
+(property "Population" "dnp" (at 83.82 109.22 0) (effects (font (size 1 1)) (hide yes)))
+(property "BOM_ID" "auxiliary_c3" (at 83.82 109.22 0) (effects (font (size 1 1)) (hide yes)))
+(pin "1")
+(pin "2")
+(instances (project "auxiliary" (path "/fd78a1d1-9bf9-50ed-9692-a93767467c7e/4d0a7c6d-5385-583b-b58d-bf025947fe80" (reference "R117") (unit 1)))) )
+(wire (pts (xy 74.93 109.22) (xy 72.39 109.22)) (stroke (width 0) (type default)))
+(global_label "AFE_SCLK_DRV" (shape passive) (at 72.39 109.22 180) (effects (font (size 1 1)) (justify right)))
+(wire (pts (xy 92.71 109.22) (xy 95.25 109.22)) (stroke (width 0) (type default)))
+(global_label "AFE_SCLK" (shape passive) (at 95.25 109.22 0) (effects (font (size 1 1)) (justify left)))
+(symbol (lib_id "RevA:R") (at 208.28 109.22 0) (unit 1) (in_bom yes) (on_board yes) (dnp yes)
+(property "Reference" "R118" (at 208.28 104.14 0) (effects (font (size 1 1))))
+(property "Value" "NOT_SELECTED" (at 208.28 106.68 0) (effects (font (size 1 1))))
+(property "Footprint" "Resistor_SMD:R_0603_1608Metric" (at 208.28 109.22 0) (effects (font (size 1 1)) (hide yes)))
+(property "Datasheet" "" (at 208.28 109.22 0) (effects (font (size 1 1)) (hide yes)))
+(property "ContractRef" "R_AFE_MOSI_SER" (at 208.28 109.22 0) (effects (font (size 1 1)) (hide yes)))
+(property "MPN" "NOT_SELECTED" (at 208.28 109.22 0) (effects (font (size 1 1)) (hide yes)))
+(property "Population" "dnp" (at 208.28 109.22 0) (effects (font (size 1 1)) (hide yes)))
+(property "BOM_ID" "auxiliary_c3" (at 208.28 109.22 0) (effects (font (size 1 1)) (hide yes)))
+(pin "1")
+(pin "2")
+(instances (project "auxiliary" (path "/fd78a1d1-9bf9-50ed-9692-a93767467c7e/4d0a7c6d-5385-583b-b58d-bf025947fe80" (reference "R118") (unit 1)))) )
+(wire (pts (xy 199.39 109.22) (xy 196.85 109.22)) (stroke (width 0) (type default)))
+(global_label "AFE_MOSI_DRV" (shape passive) (at 196.85 109.22 180) (effects (font (size 1 1)) (justify right)))
+(wire (pts (xy 217.17 109.22) (xy 219.71 109.22)) (stroke (width 0) (type default)))
+(global_label "AFE_MOSI" (shape passive) (at 219.71 109.22 0) (effects (font (size 1 1)) (justify left)))
+(symbol (lib_id "RevA:R") (at 330.2 109.22 0) (unit 1) (in_bom yes) (on_board yes) (dnp yes)
+(property "Reference" "R119" (at 330.2 104.14 0) (effects (font (size 1 1))))
+(property "Value" "NOT_SELECTED" (at 330.2 106.68 0) (effects (font (size 1 1))))
+(property "Footprint" "Resistor_SMD:R_0603_1608Metric" (at 330.2 109.22 0) (effects (font (size 1 1)) (hide yes)))
+(property "Datasheet" "" (at 330.2 109.22 0) (effects (font (size 1 1)) (hide yes)))
+(property "ContractRef" "R_AFE_CS_SER" (at 330.2 109.22 0) (effects (font (size 1 1)) (hide yes)))
+(property "MPN" "NOT_SELECTED" (at 330.2 109.22 0) (effects (font (size 1 1)) (hide yes)))
+(property "Population" "dnp" (at 330.2 109.22 0) (effects (font (size 1 1)) (hide yes)))
+(property "BOM_ID" "auxiliary_c3" (at 330.2 109.22 0) (effects (font (size 1 1)) (hide yes)))
+(pin "1")
+(pin "2")
+(instances (project "auxiliary" (path "/fd78a1d1-9bf9-50ed-9692-a93767467c7e/4d0a7c6d-5385-583b-b58d-bf025947fe80" (reference "R119") (unit 1)))) )
+(wire (pts (xy 321.31 109.22) (xy 318.77 109.22)) (stroke (width 0) (type default)))
+(global_label "AFE_CS_DRV" (shape passive) (at 318.77 109.22 180) (effects (font (size 1 1)) (justify right)))
+(wire (pts (xy 339.09 109.22) (xy 341.63 109.22)) (stroke (width 0) (type default)))
+(global_label "AFE_CS" (shape passive) (at 341.63 109.22 0) (effects (font (size 1 1)) (justify left)))
+(symbol (lib_id "RevA:R") (at 208.28 182.88 0) (unit 1) (in_bom yes) (on_board yes) (dnp yes)
+(property "Reference" "R120" (at 208.28 177.8 0) (effects (font (size 1 1))))
+(property "Value" "NOT_SELECTED" (at 208.28 180.34 0) (effects (font (size 1 1))))
+(property "Footprint" "Resistor_SMD:R_0603_1608Metric" (at 208.28 182.88 0) (effects (font (size 1 1)) (hide yes)))
+(property "Datasheet" "" (at 208.28 182.88 0) (effects (font (size 1 1)) (hide yes)))
+(property "ContractRef" "R_MCU_MISO_SER" (at 208.28 182.88 0) (effects (font (size 1 1)) (hide yes)))
+(property "MPN" "NOT_SELECTED" (at 208.28 182.88 0) (effects (font (size 1 1)) (hide yes)))
+(property "Population" "dnp" (at 208.28 182.88 0) (effects (font (size 1 1)) (hide yes)))
+(property "BOM_ID" "auxiliary_c3" (at 208.28 182.88 0) (effects (font (size 1 1)) (hide yes)))
+(pin "1")
+(pin "2")
+(instances (project "auxiliary" (path "/fd78a1d1-9bf9-50ed-9692-a93767467c7e/4d0a7c6d-5385-583b-b58d-bf025947fe80" (reference "R120") (unit 1)))) )
+(wire (pts (xy 199.39 182.88) (xy 196.85 182.88)) (stroke (width 0) (type default)))
+(global_label "MCU_MISO_DRV" (shape passive) (at 196.85 182.88 180) (effects (font (size 1 1)) (justify right)))
+(wire (pts (xy 217.17 182.88) (xy 219.71 182.88)) (stroke (width 0) (type default)))
+(global_label "MCU_MISO" (shape passive) (at 219.71 182.88 0) (effects (font (size 1 1)) (justify left)))
 )
