File: hardware/rev_a/auxiliary/auxiliary.kicad_pcb (KiCad board)
At the start: 4 copper layers, 90 x 75 mm, 52 parts, among them J101 K1_NUMBERED_SOLDER_TAILS, J102 DEVKIT_J1_NUMBERED_TAILS, J103 ADAFRUIT_5335_TAILS, J104 B6B-XH-A(LF)(SN), J105 REGULATED_5V_TAILS, J106 REMOTE_NO_STOP_CONTACT, U101 ISO7721DR, U102 TXU0304PWR, U103 TXU0304PWR, U104 TXU0304PWR, U105 TPS3703A4330DSER, U106 TPS3703A4330DSER, U107 TPS3703A5500DSER, U108 TPS3703A5500DSER, U109 SN74LVC1G97DBVR, U110 SN74LVC1G97DBVR, U111 SN74LVC2G74DCUR

Commit message: feat(hardware): complete auxiliary routing with explicit reference and cut checks
Routing:
- net MCU_3V3: track 21.7 -> 200.3 mm, vias 0 -> 14
- net BUS_OE: track 0.00 -> 103.9 mm, vias 0 -> 7
- net MCU_CLKSEL: track 0.00 -> 89.0 mm, vias 0 -> 3
- net MCU_SCLK: track 0.00 -> 85.5 mm, vias 0 -> 5
- net TARGET_VIN5: track 0.00 -> 78.8 mm, vias 0 -> 2
- net MCU_PWDN: track 0.00 -> 72.6 mm, vias 0 -> 3
- net MCU_MISO: track 0.00 -> 66.7 mm, vias 0 -> 5
- net AFE_DVDD: track 6.34 -> 72.7 mm, vias 0 -> 2
- net CONSOLE_TX: track 0.00 -> 64.1 mm, vias 0 -> 1
- net MCU_MOSI: track 0.00 -> 63.6 mm, vias 0 -> 7
- net MCU_CS: track 0.00 -> 61.6 mm, vias 0 -> 5
- net STOP_N: track 0.00 -> 57.0 mm, vias 0 -> 7
- net MCU_RESET: track 0.00 -> 54.2 mm, vias 0 -> 3
- net RAILS_OK: track 0.00 -> 50.5 mm, vias 0 -> 8
- net MCU_DRDY: track 0.00 -> 49.2 mm, vias 0 -> 4
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Other:
- board text added: "P3 CONNECTED DRAFT - NOT FOR FABRICATION"
- board text removed: "P2 PARTIAL ROUTING - NOT FOR FABRICATION"

Commit message: fix(hardware): shorten isolated clock route and refresh published handoff
Routing:
- net MCU_SCLK: track 85.5 -> 71.9 mm, vias 5 -> 4
Changed lines of the file:
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@@
 		)
 	)
-	(zone
+	(segment (start 37.700000 32.862500) (end 37.600000 31.300000) (width 0.2) (layer "F.Cu") (net 35))
+(segment (start 37.600000 31.300000) (end 38.800000 30.300000) (width 0.2) (layer "F.Cu") (net 35))
+(segment (start 38.800000 30.300000) (end 56.500000 30.000000) (width 0.2) (layer "F.Cu") (net 35))
+(segment (start 56.500000 30.000000) (end 69.800000 35.000000) (width 0.2) (layer "F.Cu") (net 35))
+(via (at 69.800000 35.000000) (size 0.6) (drill 0.3) (layers "F.Cu" "B.Cu") (net 35))
+(segment (start 69.800000 35.000000) (end 70.400000 35.600000) (width 0.2) (layer "In2.Cu") (net 35))
+(segment (start 70.400000 35.600000) (end 71.700000 37.300000) (width 0.2) (layer "In2.Cu") (net 35))
+(segment (start 71.700000 37.300000) (end 71.700000 41.400000) (width 0.2) (layer "In2.Cu") (net 35))
+(via (at 71.700000 41.400000) (size 0.6) (drill 0.3) (layers "F.Cu" "B.Cu") (net 35))
+(segment (start 71.700000 41.400000) (end 74.900000 47.300000) (width 0.2) (layer "F.Cu") (net 35))
+(segment (start 74.900000 47.300000) (end 74.800000 48.100000) (width 0.2) (layer "F.Cu") (net 35))
+(segment (start 74.800000 48.100000) (end 74.100000 49.900000) (width 0.2) (layer "F.Cu") (net 35))
+(via (at 74.100000 49.900000) (size 0.6) (drill 0.3) (layers "F.Cu" "B.Cu") (net 35))
+(segment (start 74.100000 49.900000) (end 72.100000 50.800000) (width 0.2) (layer "In2.Cu") (net 35))
+(via (at 72.100000 50.800000) (size 0.6) (drill 0.3) (layers "F.Cu" "B.Cu") (net 35))
+(segment (start 72.100000 50.800000) (end 68.900000 55.500000) (width 0.2) (layer "F.Cu") (net 35))
+(segment (start 68.900000 55.500000) (end 67.700000 57.600000) (width 0.2) (layer "F.Cu") (net 35))
+(segment (start 67.700000 57.600000) (end 67.200000 62.800000) (width 0.2) (layer "F.Cu") (net 35))
+(segment (start 67.200000 62.800000) (end 67.700000 63.500000) (width 0.2) (layer "F.Cu") (net 35))
+(segment (start 67.700000 63.500000) (end 69.400000 63.700000) (width 0.2) (layer "F.Cu") (net 35))
+(segment (start 69.400000 63.700000) (end 71.180000 65.000000) (width 0.2) (layer "F.Cu") (net 35))
+(zone
 		(net 0)
 		(net_name "")
@@
 (segment (start 54.7 32.85) (end 54.7 31.55) (width 0.2) (layer "F.Cu") (net 34))
 (via (at 54.7 31.55) (size .6) (drill .3) (layers "F.Cu" "B.Cu") (net 34))
-(segment (start 37.7 32.8625) (end 37.7 32.85) (width 0.2) (layer "F.Cu") (net 35))
-(segment (start 37.7 32.85) (end 37.6 31.7) (width 0.2) (layer "F.Cu") (net 35))
-(segment (start 37.6 31.7) (end 37.45 31.55) (width 0.2) (layer "F.Cu") (net 35))
 (segment (start 55.35 32.8625) (end 55.35 32.9) (width 0.2) (layer "F.Cu") (net 36))
 (segment (start 55.35 32.9) (end 55.35 34.15) (width 0.2) (layer "F.Cu") (net 36))
@@
 (segment (start 71.8 63.15) (end 72.55 63.65) (width 0.2) (layer "In2.Cu") (net 31))
 (segment (start 72.55 63.65) (end 73.7 65.0) (width 0.2) (layer "In2.Cu") (net 31))
-(segment (start 71.18 65.0) (end 71.2 65.0) (width 0.2) (layer "In2.Cu") (net 35))
-(segment (start 37.45 31.55) (end 37.95 31.0) (width 0.2) (layer "F.Cu") (net 35))
-(segment (start 37.95 31.0) (end 38.15 30.9) (width 0.2) (layer "F.Cu") (net 35))
-(segment (start 38.15 30.9) (end 55.3 30.45) (width 0.2) (layer "F.Cu") (net 35))
-(segment (start 55.3 30.45) (end 56.45 30.45) (width 0.2) (layer "F.Cu") (net 35))
-(segment (start 56.45 30.45) (end 69.35 35.0) (width 0.2) (layer "F.Cu") (net 35))
-(via (at 69.35 35.0) (size .6) (drill .3) (layers "F.Cu" "B.Cu") (net 35))
-(segment (start 69.35 35.0) (end 69.95 35.65) (width 0.2) (layer "In2.Cu") (net 35))
-(segment (start 69.95 35.65) (end 71.05 40.45) (width 0.2) (layer "In2.Cu") (net 35))
-(segment (start 71.05 40.45) (end 73.75 44.7) (width 0.2) (layer "In2.Cu") (net 35))
-(via (at 73.75 44.7) (size .6) (drill .3) (layers "F.Cu" "B.Cu") (net 35))
-(via (at 74.5 50.2) (size .6) (drill .3) (layers "F.Cu" "B.Cu") (net 35))
-(segment (start 74.5 50.2) (end 76.15 58.3) (width 0.2) (layer "In2.Cu") (net 35))
-(via (at 76.15 58.3) (size .6) (drill .3) (layers "F.Cu" "B.Cu") (net 35))
-(via (at 70.95 63.45) (size .6) (drill .3) (layers "F.Cu" "B.Cu") (net 35))
-(segment (start 70.95 63.45) (end 71.2 65.0) (width 0.2) (layer "In2.Cu") (net 35))
 (segment (start 10.08 32.0) (end 10.1 32.0) (width 0.2) (layer "In2.Cu") (net 26))
 (segment (start 10.1 32.0) (end 11.25 33.45) (width 0.2) (layer "In2.Cu") (net 26))
@@
 (segment (start 46.75 63.7) (end 45.8 65.0) (width 0.2) (layer "In2.Cu") (net 16))
 (segment (start 45.8 65.0) (end 45.78 65.0) (width 0.2) (layer "In2.Cu") (net 16))
-(segment (start 76.15 58.3) (end 82.7 63.7) (width 0.2) (layer "F.Cu") (net 35))
-(segment (start 82.7 63.7) (end 82.7 66.35) (width 0.2) (layer "F.Cu") (net 35))
-(segment (start 82.7 66.35) (end 79.4 66.45) (width 0.2) (layer "F.Cu") (net 35))
-(segment (start 79.4 66.45) (end 72.3 66.45) (width 0.2) (layer "F.Cu") (net 35))
-(segment (start 72.3 66.45) (end 70.95 63.45) (width 0.2) (layer "F.Cu") (net 35))
 (segment (start 59.65 46.0) (end 61.25 49.15) (width 0.3) (layer "F.Cu") (net 27))
 (segment (start 61.25 49.15) (end 62.9 49.15) (width 0.3) (layer "F.Cu") (net 27))
@@
 (segment (start 67.05 46.9) (end 68.0 46.9) (width 0.3) (layer "F.Cu") (net 27))
 (segment (start 68.0 46.9) (end 68.65 46.0) (width 0.3) (layer "F.Cu") (net 27))
-(segment (start 73.75 44.7) (end 74.6 47.45) (width 0.2) (layer "F.Cu") (net 35))
-(segment (start 74.6 47.45) (end 74.5 50.2) (width 0.2) (layer "F.Cu") (net 35))
 (segment (start 68.5 48.25) (end 68.65 47.0) (width 0.2) (layer "In2.Cu") (net 27))
 (segment (start 76.26 65.0) (end 76.25 65.0) (width 0.2) (layer "In2.Cu") (net 38))

Commit message: feat(hardware): apply the preserved five-position SPI source candidate
Apply exactly eleven manifest-verified files on 08a8ddd0, retaining
all later DNP, preservation, selection and native-fault test repairs.
The historical patch reproduces 2e50d2b; no geometry is recreated.
Five positions remain DNP/NOT_SELECTED. Native exports and copper
fills are not refreshed here. This is source publication only, not
a passing gate, approved damping value or fabrication release.
No workflow, firmware, Q1, dependency or permission setting changes
are included in this engineering commit. No project code executed
by the isolated source publisher. PR98 must remain draft.
Parts:
- added R117: NOT_SELECTED, Resistor_SMD:R_0603_1608Metric, F.Cu at (40.5, 21.3)
- added R118: NOT_SELECTED, Resistor_SMD:R_0603_1608Metric, F.Cu at (38.6, 21.3)
- added R119: NOT_SELECTED, Resistor_SMD:R_0603_1608Metric, F.Cu at (42.5, 21.3)
- added R120: NOT_SELECTED, Resistor_SMD:R_0603_1608Metric, F.Cu at (44.2, 32.2)
Connections:
- U102 pad 11: AFE_CS -> AFE_CS_DRV
- U102 pad 12: AFE_MOSI -> AFE_MOSI_DRV
- U102 pad 13: AFE_SCLK -> AFE_SCLK_DRV
- U102 pad 5: MCU_MISO -> MCU_MISO_DRV
Routing:
- net AFE_CS: track 22.8 -> 12.5 mm
- net AFE_CS_DRV: track 0.00 -> 8.72 mm, vias 0 -> 2
- net AFE_MOSI: track 22.6 -> 13.9 mm
- net AFE_MOSI_DRV: track 0.00 -> 7.93 mm, vias 0 -> 2
- net AFE_SCLK_DRV: track 0.00 -> 6.64 mm, vias 0 -> 2
- net AFE_SCLK: track 26.5 -> 20.2 mm, vias 3 -> 2
- net MCU_MISO_DRV: track 0.00 -> 5.29 mm, vias 0 -> 2
- net MCU_MISO: track 66.7 -> 65.4 mm, vias 5 -> 4

Commit message: fix(hardware): declare SPI nets before pads and import native exports
Actual KiCad9.0.2 diagnosed five driver pads loading as no-net because
their declarations appeared after footprints. Move only declarations;
retain numeric nets, pad fields and planar routes. Remove exactly two
native-DRC single-layer via stubs and extend only the explicit L5 delta.
Use genuine native XML/CSV from immutable source27c6525d/run38074668398.
Reconcile exact inventory increases, preserving all mutation loops.
One AST-preserving formatter fix. Fourteen files, independently fixed
expected treebd59a0c. No original snapshot, firmware, Q1, workflow or
dependency/gate changes. Installed-pytest338 focused passes locally;
not a locked or native correction pass. Fresh native refill/faults
and K2 binding/access review remain. No fabrication or power release.
Routing:
- net MCU_MISO: vias 4 -> 3
- net AFE_SCLK: vias 2 -> 1
